File: Control Systems.kicad_sch (KiCad schematic)
At the start: 13 parts, among them SW1 SW_SPDT, U1 STM32F446RETx

Commit message: Test branch
Parts:
- removed SW1: SW_SPDT, symbol Switch:SW_SPDT
Changed lines of the file:
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@@
 (kicad_sch
-	(version 20231120)
+	(version 20250114)
 	(generator "eeschema")
-	(generator_version "8.0")
+	(generator_version "9.0")
 	(paper "A4")
+	(text "NRST\n"
+		(exclude_from_sim no)
+		(at 124.714 51.308 0)
+		(effects
+			(font
+				(size 1.27 1.27)
+			)
+		)
+	)
+	(text "SW_BOOT0\n"
+		(exclude_from_sim no)
+		(at 116.332 56.642 0)
+		(effects
+			(font
+				(size 0.762 0.762)
+			)
+		)
+	)
+	(text "BOOT0\n"
+		(exclude_from_sim no)
+		(at 129.286 56.642 0)
+		(effects
+			(font
+				(size 0.762 0.762)
+			)
+		)
+	)
+	(text_box "GND = run code 3.3V = run bootloader to flash new code\n"
+		(exclude_from_sim no)
+		(at 99.06 64.77 0)
+		(size 19.05 8.89)
+		(margins 0.9525 0.9525 0.9525 0.9525)
+		(stroke
+			(width 0)
+			(type default)
+		)
+		(fill
+			(type none)
+		)
+		(effects
+			(font
+				(size 1.27 1.27)
+			)
+			(justify left top)
+		)
+	)
+	(text_box "NRST reset when low and run when high, has internal pullup, put 100nf capacitor to prevent sprurious reset"
+		(exclude_from_sim no)
+		(at 57.15 54.61 0)
+		(size 26.67 11.43)
+		(margins 0.9525 0.9525 0.9525 0.9525)
+		(stroke
+			(width 0)
+			(type default)
+		)
+		(fill
+			(type none)
+		)
+		(effects
+			(font
+				(size 1.27 1.27)
+			)
+			(justify left top)
+		)
+	)
 	(junction
 		(at 92.71 45.72)
@@
 			(width 0)
 			(type default)
-		)
-	)
-	(text_box "GND = run code 3.3V = run bootloader to flash new code\n"
-		(exclude_from_sim no)
-		(at 99.06 64.77 0)
-		(size 19.05 8.89)
-		(stroke
-			(width 0)
-			(type default)
-		)
-		(fill
-			(type none)
-		)
-		(effects
-			(font
-				(size 1.27 1.27)
-			)
-			(justify left top)
-		)
-	)
-	(text_box "NRST reset when low and run when high, has internal pullup, put 100nf capacitor to prevent sprurious reset"
-		(exclude_from_sim no)
-		(at 57.15 54.61 0)
-		(size 26.67 11.43)
-		(stroke
-			(width 0)
-			(type default)
-		)
-		(fill
-			(type none)
-		)
-		(effects
-			(font
-				(size 1.27 1.27)
-			)
-			(justify left top)
-		)
-	)
-	(text "NRST\n"
-		(exclude_from_sim no)
-		(at 124.714 51.308 0)
-		(effects
-			(font
-				(size 1.27 1.27)
-			)
-		)
-	)
-	(text "SW_BOOT0\n"
-		(exclude_from_sim no)
-		(at 116.332 56.642 0)
-		(effects
-			(font
-				(size 0.762 0.762)
-			)
-		)
-	)
-	(text "BOOT0\n"
-		(exclude_from_sim no)
-		(at 129.286 56.642 0)
-		(effects
-			(font
-				(size 0.762 0.762)
-			)
 		)
 	)
@@
 	)
 	(symbol
-		(lib_id "Switch:SW_SPDT")
-		(at 107.95 57.15 180)
-		(unit 1)
-		(exclude_from_sim no)
-		(in_bom yes)
-		(on_board yes)
-		(dnp no)
-		(property "Reference" "SW1"
-			(at 107.442 66.04 0)
-			(effects
-				(font
-					(size 1.27 1.27)
-				)
-				(hide yes)
-			)
-		)
-		(property "Value" "SW_SPDT"
-			(at 107.696 62.992 0)
-			(effects
-				(font
-					(size 1.27 1.27)
-				)
-			)
-		)
-		(property "Footprint" ""
-			(at 107.95 57.15 0)
-			(effects
-				(font
-					(size 1.27 1.27)
-				)
-				(hide yes)
-			)
-		)
-		(property "Datasheet" "~"
-			(at 107.95 49.53 0)
-			(effects
-				(font
-					(size 1.27 1.27)
-				)
-				(hide yes)
-			)
-		)
-		(property "Description" "Switch, single pole double throw"
-			(at 107.95 57.15 0)
-			(effects
-				(font
-					(size 1.27 1.27)
-				)
-				(hide yes)
-			)
-		)
-		(pin "3"
-		)
-		(pin "2"
-		)
-		(pin "1"
-		)
-		(instances
-			(project ""
-				(path "/31c0570c-1cf3-4765-824d-7a8db7e67b19"
-					(reference "SW1")
-					(unit 1)
-				)
-			)
-		)
-	)
-	(symbol
 		(lib_id "Device:C")
 		(at 82.55 39.37 0)
@@
 		)
 	)
+	(embedded_fonts no)
 )
