File: Control Systems.kicad_sch (KiCad schematic)
At the start: 34 parts, among them IC1 LM66200DRLR, J1 XT60-M, J2 47346-0001, J3 61300311121, J4 61300311121, J5 61300311121, J6 61300311121, J7 Conn_01x04_Pin, J8 SD_Card_Receptacle, U1 STM32F446RETx, U2 ICM-20948, U3 BMI088, U4 NEO-M8N-0, U5 MMC5983MA, U6 TL1963A-33DCYR, Y1 SIT8924BA-20.0

Commit message: test
Connections:
- net SPI2_CS: now reaches U1.55 (PB3)
- net SPI2_NSS renamed SPI2_CS_2
Other:
- moved on the sheet: A1, U4
Changed lines of the file:
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@@
 	(wire
 		(pts
-			(xy 139.7 161.29) (xy 139.7 172.72)
+			(xy 137.16 161.29) (xy 137.16 172.72)
 		)
 		(stroke
@@
 	(wire
 		(pts
+			(xy 254 199.39) (xy 267.97 199.39)
+		)
+		(stroke
+			(width 0)
+			(type default)
+		)
+	)
+	(wire
+		(pts
 			(xy 200.66 189.23) (xy 213.36 189.23)
 		)
@@
 	(wire
 		(pts
+			(xy 137.16 161.29) (xy 139.7 161.29)
+		)
+		(stroke
+			(width 0)
+			(type default)
+		)
+	)
+	(wire
+		(pts
 			(xy 363.22 40.64) (xy 367.03 40.64)
 		)
@@
 	(wire
 		(pts
+			(xy 137.16 172.72) (xy 139.7 172.72)
+		)
+		(stroke
+			(width 0)
+			(type default)
+		)
+	)
+	(wire
+		(pts
 			(xy 313.69 35.56) (xy 327.66 35.56)
 		)
@@
 		)
 	)
+	(label "SPI2_CS"
+		(at 256.54 199.39 0)
+		(effects
+			(font
+				(size 0.889 0.889)
+			)
+			(justify left bottom)
+		)
+	)
 	(label "XTAL_IN"
 		(at 161.29 166.37 0)
@@
 		)
 	)
-	(label "SPI2_NSS"
+	(label "SPI2_CS_2"
 		(at 255.27 201.93 0)
 		(effects
@@
 	(symbol
 		(lib_id "NEO-M8N-0:NEO-M8N-0")
-		(at 369.57 154.94 0)
+		(at 332.74 156.21 0)
 		(unit 1)
 		(exclude_from_sim no)
@@
 		(fields_autoplaced yes)
 		(property "Reference" "U4"
-			(at 369.57 127 0)
+			(at 332.74 128.27 0)
 			(effects
 				(font
@@
 		)
 		(property "Value" "NEO-M8N-0"
-			(at 369.57 129.54 0)
+			(at 332.74 130.81 0)
 			(effects
 				(font
@@
 		)
 		(property "Footprint" "NEO-M8N-0:XCVR_NEO-M8N-0"
-			(at 369.57 154.94 0)
+			(at 332.74 156.21 0)
 			(effects
 				(font
@@
 		)
 		(property "Datasheet" ""
-			(at 369.57 154.94 0)
+			(at 332.74 156.21 0)
 			(effects
 				(font
@@
 		)
 		(property "Description" ""
-			(at 369.57 154.94 0)
+			(at 332.74 156.21 0)
 			(effects
 				(font
@@
 		)
 		(property "PARTREV" "R04"
-			(at 369.57 154.94 0)
+			(at 332.74 156.21 0)
 			(effects
 				(font
@@
 		)
 		(property "MF" "U-Blox America"
-			(at 369.57 154.94 0)
+			(at 332.74 156.21 0)
 			(effects
 				(font
@@
 		)
 		(property "STANDARD" "Manufacturer Recommendation"
-			(at 369.57 154.94 0)
+			(at 332.74 156.21 0)
 			(effects
 				(font
@@
 	(symbol
 		(lib_id "MS561101BA03-50:MS561101BA03-50")
-		(at 308.61 100.33 0)
+		(at 287.02 91.44 0)
 		(unit 1)
 		(exclude_from_sim no)
@@
 		(fields_autoplaced yes)
 		(property "Reference" "A1"
-			(at 308.61 85.09 0)
+			(at 287.02 76.2 0)
 			(effects
 				(font
@@
 		)
 		(property "Value" "MS561101BA03-50"
-			(at 308.61 87.63 0)
+			(at 287.02 78.74 0)
 			(effects
 				(font
@@
 		)
 		(property "Footprint" "MS561101BA03-50:XDCR_MS561101BA03-50"
-			(at 308.61 100.33 0)
+			(at 287.02 91.44 0)
 			(effects
 				(font
@@
 		)
 		(property "Datasheet" ""
-			(at 308.61 100.33 0)
+			(at 287.02 91.44 0)
 			(effects
 				(font
@@
 		)
 		(property "Description" ""
-			(at 308.61 100.33 0)
+			(at 287.02 91.44 0)
 			(effects
 				(font
@@
 		)
 		(property "PARTREV" "06/2017"
-			(at 308.61 100.33 0)
+			(at 287.02 91.44 0)
 			(effects
 				(font
@@
 		)
 		(property "STANDARD" "Manufacturer Recommendations"
-			(at 308.61 100.33 0)
+			(at 287.02 91.44 0)
 			(effects
 				(font
@@
 		)
 		(property "MAXIMUM_PACKAGE_HEIGHT" "1.1mm"
-			(at 308.61 100.33 0)
+			(at 287.02 91.44 0)
 			(effects
 				(font
@@
 		)
 		(property "MANUFACTURER" "TE Connectivity"
-			(at 308.61 100.33 0)
+			(at 287.02 91.44 0)
 			(effects
 				(font

Commit message: Finished all sensors, added LDO, and GPS wiring
Parts:
- removed J8: SD_Card_Receptacle, symbol Connector:SD_Card_Receptacle
- removed U2: ICM-20948, Sensor_Motion:InvenSense_QFN-24_3x3mm_P0.4mm, symbol Sensor_Motion:ICM-20948
- added C15, C16, C21: 100n, symbol Device:C
- added C17: 10uf, symbol Device:C
- added C18: 100nf, symbol Device:C
- added C19: 10nf, symbol Device:C
- added C20: 10u, symbol Device:C
- added C22, C23: 2u2, symbol Device:C
- added D1, D2, D3, D4, D5, D6: ESD9B3.3ST5G, Diode_SMD:D_SOD-923, symbol Diode:ESD9B3.3ST5G
- added D10, D11, D8, D9: TVS, Diode_SMD:Nexperia_DSN1608-2_1.6x0.8mm, symbol Diode:PTVS10VZ1USK
- added FB1: 120R, symbol Device:FerriteBead
- added J10: Canbus, symbol Connector:Screw_Terminal_01x02
- added J11: Conn_01x09_Socket, symbol Connector:Conn_01x09_Socket
- added J12: Conn_01x05_Socket, symbol Connector:Conn_01x05_Socket
- added J13: GPIO_terminals, symbol Connector:Screw_Terminal_01x07
- added J8: MEM2061-01-188-00-A_REVA, MEM2061-01-188-00-A_REVA:GCT_MEM2061-01-188-00-A_REVA, symbol MEM2061-01-188-00-A_REVA:MEM2061-01-188-00-A_REVA
- added J9: 5-1814832-2, 5-1814832-2:TE_5-1814832-2, symbol 5-1814832-2:5-1814832-2
- added L1: 27nH, symbol Device:L
- added R10, R11, R4, R7, R8, R9: 47k, symbol Device:R
- added R12: 56k, symbol Device:R
- added R5: 4k7, symbol Device:R
- added R6: 10, symbol Device:R
- added U2: LSM6DSL, Package_LGA:LGA-14_3x2.5mm_P0.5mm_LayoutBorder3x4y, symbol Sensor_Motion:LSM6DSL
- added U7: TPS552882QWRPMRQ1, TPS552882QWRPMRQ1:CONV_TPS552882QWRPMRQ1, symbol TPS552882QWRPMRQ1:TPS552882QWRPMRQ1
- added U8: USBLC6-2SC6, Package_TO_SOT_SMD:SOT-23-6, symbol Power_Protection:USBLC6-2SC6
Connections:
- net +3.3V: now also A1.1 (VDD), U4.22 (V_BCKP), U4.23 (VCC), C15.1, C16.1, C17.1, C18.1, C20.1, C21.1, J11.1 (Pin_1), J8.4 (VDD), R10.1, R11.1, R12.2, R4.1, R5.1, R7.1, R8.1, R9.1, U2.5 (VDDIO), U2.8 (VDD); no longer J3.2, J4.2, J5.2, J6.2
- net CAN2_RX: now also J10.1 (Pin_1)
- net CAN2_TX: now also J10.2 (Pin_2)
- net GND: now also J3.3, J4.3, J5.3, J6.3, C20.2, D1.1 (A1), D10.2 (A), D11.2 (A), D2.1 (A1), D3.1 (A1), D4.1 (A1), D5.1 (A1), D6.1 (A1), D8.2 (A), D9.2 (A), J8.10 (CD2), J8.11 (GND), J8.12 (GND__1), J8.6 (VSS)
- net I2C1_SCL: now also R5.2
- net I2C1_SDA: now also R4.2
- net SPI1_MISO: now also J11.6 (Pin_6)
- net SPI1_MOSI: now also J11.7 (Pin_7)
- net SPI1_SCK: now also J11.5 (Pin_5)
- net SPI2_CS: now also A1.4 (~{CSB})
- net SPI2_CS_2: now also U4.18 (SDA/SPI_CS_N)
- net SPI2_MISO: now also A1.6 (SDO)
- net SPI2_MOSI: now also A1.7 (SDI/SDA)
- net at U4.10 (GND): now also U4.12 (GND__1), U4.13 (GND__2), U4.24 (GND__3)
- net RF_IN: now reaches U4.11 (RF_IN)
- net RF_IN: now also J9.1, L1.1
- net GPS_SPI2_CLK: now reaches U4.19 (SCL/SPI_CLK)
- net GPS_SPI2_MISO: now reaches U4.20 (TXD/SPI_MISO)
- net GPS_SPI2_MOSI: now reaches U4.21 (RXD/SPI_MOSI)
- net at U4.9 (VCC_RF): now also R6.1
- net at U6.1 (IN): now also IC1.2 (VOUT@1), IC1.7 (VOUT@2); no longer J1.P (POS)
- net at U6.2 (GND_2): now also U6.4 (GND_4)
- net at A1.3 (GND): now also C21.2
- net SPI2_CLK: now reaches A1.8 (SCLK)
- net at IC1.3 (VIN1): now also J1.P (POS)
- net at IC1.4 (ON): now also IC1.5 (GND@2)
- net at IC1.6 (VIN2): now also C23.1, FB1.2
- net GPIO_2: now reaches U1.11 (PC3)
- net GPIO_2: now also J13.2 (Pin_2)
- net RADIO_RST: now reaches U1.2 (PC13)
- net RADIO_RST: now also J11.9 (Pin_9)
- net SPI1_CS: now reaches U1.24 (PC4)
- net SPI1_CS_2: now reaches U1.25 (PC5)
- net SPI1_CS_2: now also J11.8 (Pin_8)
- net SDIO_CK: now reaches U1.28 (PB2)
- net SDIO_CK: now also D6.2 (A2), J8.5 (CLK), R11.2
- net RADIO_G1: now reaches U1.3 (PC14)
- net RADIO_G1: now also J12.5 (Pin_5)
- net GPIO_7: now reaches U1.36 (PB15)
- net GPIO_7: now also J13.7 (Pin_7)
- net SDIO_D0: now reaches U1.39 (PC8)
- net SDIO_D0: now also D1.2 (A2), J8.7 (DAT0)
- net RADIO_G0: now reaches U1.4 (PC15)
- net RADIO_G0: now also J11.4 (Pin_4)
- net SDIO_NCD: now reaches U1.41 (PA8)
- net GPIO_4: now reaches U1.50 (PA15)
- net GPIO_4: now also J13.4 (Pin_4)
- net SDIO_D2: now reaches U1.51 (PC10)
- net SDIO_D2: now also D3.2 (A2), J8.1 (DAT2), R8.2
- net SDIO_D3: now reaches U1.52 (PC11)
- net SDIO_D3: now also D4.2 (A2), J8.2 (CD/DAT3), R9.2
- net GPIO_3: now reaches U1.53 (PC12)
- net GPIO_3: now also J13.3 (Pin_3)
- net SDIO_CMD: now reaches U1.54 (PD2)
- net SDIO_CMD: now also D5.2 (A2), J8.3 (CMD), R10.2
- net GPIO_5: now reaches U1.57 (PB5)
- net GPIO_5: now also J13.5 (Pin_5)
- net GPIO_6: now reaches U1.59 (PB7)
- net GPIO_6: now also J13.6 (Pin_6)
- net GPIO_1: now reaches U1.8 (PC0)
- net GPIO_1: now also J13.1 (Pin_1)
- net at J2.2 (D-): now also U8.3 (I/O2)
- net at J2.3 (D+): now also U8.1 (I/O1)
- net at J2.5 (GND): now also C22.2, C23.2, U8.5 (VBUS)
- net GPIO_14 renamed RADIO_EN
- net RADIO_EN: now also J11.3 (Pin_3)
- net GPIO_9C renamed SDIO_D1
- net SDIO_D1: now also D2.2 (A2), J8.8 (DAT1), R7.2
- net VBUS renamed +VBUS
- net +VBUS: now also C22.1, FB1.1, U8.2 (GND)
- new net: U2.6 (GND), U2.7 (GND)
- new net: C19.1, L1.2, R6.2
- new net: C17.2, C18.2
- new net: J9.S1, J9.S2, J9.S3, J9.S4
- new net 8.2V: D10.1 (K), D11.1 (K), D8.1 (K), D9.1 (K), J3.2, J4.2, J5.2, J6.2
- new net LSM_I2C_SCL: U2.13 (SCL)
- new net LSM_I2C_SDA: U2.14 (SDA)
- new net SD_NCD: J8.9 (CD1), R12.1
- no-connect marks 1 -> 9
Other:
- note added: "Adafruit RFM69HCW"
- note added: "I DONT CARE ANYMORE IM JUST PROVIDING POWER FOR 2 SERVOS AHHHHHH FUCK THIS DUDE"
- note added: "REVIEW THIS VCC DIAGRAM"
- note added: "SD CARD receptacle"
- note added: "VERIFY PI FILTER AND TVS DIODE"
- note removed: "Finish Pi filter or other filter and TVS diode"
- moved on the sheet: A1, C1, C2, C3, C4, C5, C6, C7, C8, IC1, J1, J2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

Commit message: Feat: Finished voltage regulator and interupts
Parts:
- removed IC1: LM66200DRLR, LM66200DRLR:SOT8, symbol LM66200DRLR:LM66200DRLR
- removed J11: Conn_01x09_Socket, symbol Connector:Conn_01x09_Socket
- removed J12: Conn_01x05_Socket, symbol Connector:Conn_01x05_Socket
- removed J13: GPIO_terminals, symbol Connector:Screw_Terminal_01x07
- added C24, C34, C35: 100n, symbol Device:C_Small
- added C25: 2.2n, symbol Device:C_Small
- added C26: 15p, symbol Device:C_Small
- added C27: 4.7u, symbol Device:C_Small
- added C28, C33: 1u, symbol Device:C_Small
- added C29, C32: 22u, symbol Device:C_Small
- added C30: 270u, symbol Device:C_Polarized_Small_US
- added C31: 180u, symbol Device:C_Polarized_Small_US
- added D12, D13, D14, D7: SMAJ6.0CA, Diode_SMD:D_SMA, symbol Diode:SMAJ6.0CA
- added D15: TVS, Diode_SMD:Nexperia_DSN1608-2_1.6x0.8mm, symbol Diode:PTVS10VZ1USK
- added J11: Canbus, symbol Connector:Screw_Terminal_01x03
- added J14, J15: Conn_01x08_Socket, symbol Connector:Conn_01x08_Socket
- added L2: 5.6u, symbol Device:L
- added Q1, Q2: CSD18504Q5A, Package_TO_SOT_SMD:TDSON-8-1, symbol Transistor_FET:CSD18504Q5A
- added R13: 80k, symbol Device:R
- added R14: 50k, symbol Device:R_Small
- added R15: 30.1k, symbol Device:R_Small
- added R16: 133k, symbol Device:R_Small
- added R17, R20: 100k, symbol Device:R_Small
- added R18: 16k, symbol Device:R_Small
- added R19: 383k, symbol Device:R_Small
- added R21, R22: 4.7, symbol Device:R_Small
- added R23, R24: 102k, symbol Device:R_Small
- added U10: TPS2121RUXR, TPS2121RUXR:IC_TPS2121RUXR, symbol TPS2121RUXRr:TPS2121RUXR
- J10: value Canbus -> Battery input
Connections:
- net ADC1_IN1 is gone; now on net GPIO_EXTI1: U1.15 (PA1)
- net ADC1_INO is gone; now on net GPIO_EXTI0: U1.14 (PA0)
- net ADC_IN2 is gone; now on net GPIO_EXTI2: U1.16 (PA2)
- net ADC_IN3 is gone; now on net GPIO_EXTI3: U1.17 (PA3)
- net GPIO_9 is gone; now on net GNSS_GPIO: U1.42 (PA9)
- net IMU_MOSI is gone; now on net I2C1_SDA: U3.9 (SDA/SDI)
- net IMU_SCK is gone; now on net I2C1_SCL: U3.8 (SCL/SCK)
- net USB_OTG_DM is gone; now on net USB_D_N: U1.44 (PA11)
- net USB_OTG_DP is gone; now on net USB_D_P: U1.45 (PA12)
- net +3.3V: now also U6.3 (OUT), J14.5 (Pin_5); no longer U1.1 (VBAT), U1.13 (VDDA), U1.19 (VDD), U1.32 (VDD), U1.48 (VDD), U1.64 (VDD)
- net CAN2_RX: now also J11.1 (Pin_1); no longer J10.1 (Pin_1)
- net CAN2_TX: now also J11.2 (Pin_2); no longer J10.2 (Pin_2)
- net GND: now also D12.2 (A2), D13.2 (A2), D14.2 (A2), D7.2 (A2)
- net PWM_TIM3_CH1: now also D7.1 (A1)
- net PWM_TIM3_CH2: now also D12.1 (A1)
- net PWM_TIM3_CH3: now also D13.1 (A1)
- net PWM_TIM3_CH4: now also D14.1 (A1)
- net RADIO_RST: now also J15.6 (Pin_6)
- net SPI1_CS_2: now also J15.5 (Pin_5)
- net SPI1_MISO: now also J15.2 (Pin_2)
- net SPI1_MOSI: now also J15.3 (Pin_3)
- net SPI1_SCK: now also J15.4 (Pin_4)
- net GPIO_EXTI3: now reaches U2.4 (INT1)
- net GPIO_EXTI2: now reaches U5.15 (INT)
- net at C1.1, C2.1, C3.1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: now also U1.1 (VBAT), U1.13 (VDDA), U1.19 (VDD), U1.32 (VDD), U1.48 (VDD), U1.64 (VDD)
- net GNSS_GPIO: now reaches U4.4 (EXTINT)
- net at U6.1 (IN): now also U10.1 (OUT), U10.1_1 (OUT), U10.8 (OUT), U10.8_1 (OUT)
- net VIN_7.4V: now reaches J1.P (POS)
- net VIN_7.4V: now also U7.3 (VIN), C31.1, C32.1, C33.1, D15.1 (K), Q1.5 (D), R19.1
- net at C23.1, FB1.2: now also U10.2 (IN2), U10.2_1 (IN2)
- net at U7.1 (DR1L): now also R22.2
- net at U7.10 (AGND): now also U7.24 (PGND__1), U7.9 (PGND), Q2.1 (S), Q2.2 (S), Q2.3 (S), R15.1
- net +8.2V: now reaches U7.11 (VOUT)
- net +8.2V: now also U7.12 (ISP), U7.13 (ISN), U7.26 (VOUT__1), C28.1, C29.1, C30.1, R17.1
- net SWR_FB: now reaches U7.14 (FB)
- net SWR_FB: now also R17.2, R18.1
- net at U7.15 (MODE): now also U7.7 (DITH/SYNC), C26.2, R14.2, R16.2
- net at U7.17 (ILIM): now also R15.2
- net at U7.18 (COMP): now also C25.1, C26.1
- net at U7.19 (VCC): now also C27.1
- net at U7.2 (DR1H): now also R21.2
- net SWR_BOOT2: now reaches U7.20 (BOOT2)
- net SWR_BOOT2: now also C35.2
- net at U7.21 (SW2): now also U7.25 (SW2__1), C35.1, L2.2
- net SWR_BOOT1: now reaches U7.22 (BOOT1)
- net SWR_BOOT1: now also C34.1
- net at U7.23 (SW1): now also C34.2, L2.1, Q1.1 (S), Q1.2 (S), Q1.3 (S), Q2.5 (D)
- net SWR_EN: now reaches U7.4 (EN/UVLO)
- net SWR_EN: now also R19.2, R20.1
- net at U7.5 (PG): now also R24.1
- net at U7.6 (~{CC}): now also R23.1
- net at U7.8 (FSW): now also R14.1
- net GPIO_EXTI1: now reaches U3.12 (INT3)
- net GPIO_EXTI0: now reaches U3.16 (INT1)
- net USB_D_N: now reaches U8.4 (I/O2)
- net USB_D_P: now reaches U8.6 (I/O1)
- net GPIO_1: no longer names the net of U1.8 (PC0)
- net GPIO_2: no longer names the net of U1.11 (PC3)
- net GPIO_3 renamed RADIO_D5
- net RADIO_D5: now also J15.7 (Pin_7)
- net GPIO_4: no longer names the net of U1.50 (PA15)
- net GPIO_5: no longer names the net of U1.57 (PB5)
- net GPIO_6: no longer names the net of U1.59 (PB7)
- net GPIO_7: no longer names the net of U1.36 (PB15)
- net RADIO_G0 renamed RADIO_D0
- net RADIO_D0: now also J14.6 (Pin_6)
- net RADIO_G1 renamed RADIO_D4
- net RADIO_D4: now also J14.4 (Pin_4)
- net SPI1_NSS renamed CAN_INT
- net CAN_INT: now also J11.3 (Pin_3)
- new net: Q1.4 (G), R21.1
- new net: Q2.4 (G), R22.1
- new net: R23.2, R24.2
- new net: C24.1, U10.11 (SS)
- new net: C28.2, C29.2, C30.2, R18.2
- new net: C25.2, R16.1
- new net: C31.2, C32.2, C33.2, R20.2
- new net: R13.1, U10.10 (ILIM)
- new net: U10.12 (GND), U10.9 (ST)
- new net: U10.3 (CP2), U10.4 (OV2), U10.5 (OV1), U10.6 (PR1)
- new net: J10.2 (Pin_2), U10.7 (IN1), U10.7_1 (IN1)
- no-connect marks 9 -> 15
Other:
- note added: "4.1.2 of DTEG IREC RULES: States that tracking elements (GPS) must be powered seperatly So added a second screw terminal for just PCB power can be 3.7-7.4V"
- note added: "NEED A DIFFERENT POWER SOURCE FOR PCB VS MOTORS"
- note added: "TODO: Need an LED FOR POWER, RX & TX, and general LED Need high side switch for servos"
- note added: "Verify PINOUT for STM"
- note removed: "Adafruit RFM69HCW"
- note removed: "Switching diode for USB & battery power"
- moved on the sheet: A1, C1, C2, C21, C22, C23, C3, C4, C5, C6, C7, FB1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

Commit message: feat: minor changes and updates to schematic
Parts:
- removed J7: Conn_01x04_Pin, symbol Connector:Conn_01x04_Pin
- added C36: 310n, symbol Device:C_Small
- added D16: RED, symbol Device:LED
- added D17, D18: Green, symbol Device:LED
- added D19: TVS, Diode_SMD:Nexperia_DSN1608-2_1.6x0.8mm, symbol Diode:PTVS10VZ1USK
- added D20: ESD9B3.3ST5G, Diode_SMD:D_SOD-923, symbol Diode:ESD9B3.3ST5G
- added J12: Conn_02x03_Odd_Even, symbol Connector_Generic:Conn_02x03_Odd_Even
- added J7: GPIO, symbol Connector:Screw_Terminal_01x03
- added R25, R26, R27: 1K, symbol Device:R_Small
- added U9: TPS1H200AQDGNRQ1, TPS1H200AQDGNRQ1:SOP65P490X110-9N, symbol TPS1H200AQDGNRQ1:TPS1H200AQDGNRQ1
Connections:
- net GPS_SPI2_CLK is gone; now on net SPI2_SCK: U4.19 (SCL/SPI_CLK)
- net GPS_SPI2_MISO is gone; now on net SPI2_MISO: U4.20 (TXD/SPI_MISO)
- net GPS_SPI2_MOSI is gone; now on net SPI2_MOSI: U4.21 (RXD/SPI_MOSI)
- net IMU_MISO is gone; now on net SPI1_MISO: U3.10 (SDO2), U3.15 (SDO1)
- net LSM_I2C_SCL is gone; now on net I2C1_SCL: U2.13 (SCL)
- net LSM_I2C_SDA is gone; now on net I2C1_SDA: U2.14 (SDA)
- net MAG_I2C1_SCL is gone; now on net I2C1_SCL: U5.1 (SCL/SPI_SCK)
- net MAG_I2C1_SDA is gone; now on net I2C1_SDA: U5.16 (SDA/SPI_SDI)
- net SPI2_CLK is gone; now on net SPI2_SCK: A1.8 (SCLK)
- net +3.3V: now also D16.2 (A), D20.2 (A2), J12.2 (Pin_2)
- net +8.2V: now also U9.8 (VS)
- net GND: now also D20.1 (A1), J12.4 (Pin_4), J12.6 (Pin_6), R26.2
- net I2C1_SCL: no longer U3.8 (SCL/SCK)
- net I2C1_SDA: no longer U3.9 (SDA/SDI)
- net MCU_NRST: now also J12.5 (Pin_5)
- net SPI1_CS: now also U3.14 (CSB1)
- net SPI1_MOSI: now also U3.9 (SDA/SDI)
- net SPI1_SCK: now also U3.8 (SCL/SCK)
- net SYS_SWCLK: now also J12.3 (Pin_3)
- net SYS_SWDIO: now also J12.1 (Pin_1)
- net at C27.1, U7.19 (VCC): now also R24.1, U7.5 (PG)
- net at C12.2: now also C11.2
- net at U6.2 (GND_2), U6.4 (GND_4): now also R25.2
- net SPI1_CS_3: now reaches U3.5 (CSB2)
- net SPI1_CS_3: now also U1.59 (PB7)
- net at J10.2 (Pin_2), U10.7 (IN1), U10.7_1 (IN1): now also D19.1 (K)
- net at J10.1 (Pin_1): now also D19.2 (A)
- net GPIO_1: now reaches U1.11 (PC3)
- net GPIO_1: now also J7.1 (Pin_1)
- net GP_LED: now reaches U1.36 (PB15)
- net GP_LED: now also D17.1 (K), D17.2 (A), R26.1
- net RX_LED: now reaches U1.50 (PA15)
- net RX_LED: now also D18.1 (K), D18.2 (A), R27.1
- net GPIO_2: now reaches U1.57 (PB5)
- net GPIO_2: now also J7.2 (Pin_2)
- net Servo_HS_Sw: now reaches U1.8 (PC0)
- net Servo_HS_Sw: now also U9.1 (IN)
- net 8.2V renamed Servo +8.2V
- net Servo +8.2V: now also U9.7 (OUT)
- net RADIO_EN renamed GPIO_3
- net GPIO_3: now also J7.3 (Pin_3)
- new net: C36.2, U9.2 (DIAG_EN)
- new net: U9.4 (CL), U9.6 (GND)
- new net: C36.1, U9.5 (DELAY)
- new net PWR_LED_K: D16.1 (K), R25.1
- no-connect marks 15 -> 23
Other:
- note added: "433mHz LORA radio"
- note added: "High Side switch no current limiting"
- note removed: "Figure out SWD wiring"
- note removed: "NEED A DIFFERENT POWER SOURCE FOR PCB VS MOTORS"
- note removed: "TODO: Need an LED FOR POWER, RX & TX, and general LED Need high side switch for servos"
- moved on the sheet: D7
